File: logic_tester.kicad_pcb (KiCad board)
At the start: 2 copper layers, 36 parts, among them J1 15EDGR-3.5-02P, U1 LM339D, U2 LM317MDT

Commit message: Geo reannotate
Parts:
- renumbered C4 to C1, C2 to C10, C5 to C2, C6 to C3, C9 to C4, C7 to C5, C10 to C6, C3 to C7, C1 to C8, C8 to C9, D5 to D3, D3 to D4, R11 to R1, R4 to R10, R9 to R11, R2 to R12, R14 to R13, R20 to R14, R10 to R15, R18 to R16, R15 to R17, R17 to R18, R16 to R19, R12 to R2, R13 to R3, R6 to R4, R7 to R5, R8 to R6, R1 to R7, R5 to R8, R3 to R9
Changed lines of the file:
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@@
     (zone_connect 1)
     (attr smd)
-    (fp_text reference "C8" (at 0 -1.3) (layer "F.SilkS") hide
+    (fp_text reference "C9" (at 0 -1.3) (layer "F.SilkS") hide
         (effects (font (size 0.8 0.8) (thickness 0.15)))
     )
@@
     (property "ki_keywords" "R res resistor")
     (attr smd)
-    (fp_text reference "R4" (at 0 -1.3) (layer "F.SilkS")
+    (fp_text reference "R10" (at 0 -1.3) (layer "F.SilkS")
         (effects (font (size 0.8 0.8) (thickness 0.15)))
     )
@@
     (property "ki_keywords" "R res resistor")
     (attr smd)
-    (fp_text reference "R5" (at 0 -1.3) (layer "F.SilkS")
+    (fp_text reference "R8" (at 0 -1.3) (layer "F.SilkS")
         (effects (font (size 0.8 0.8) (thickness 0.15)))
     )
@@
     (property "ki_keywords" "R res resistor")
     (attr smd)
-    (fp_text reference "R10" (at 0 -1.3) (layer "F.SilkS")
+    (fp_text reference "R15" (at 0 -1.3) (layer "F.SilkS")
         (effects (font (size 0.8 0.8) (thickness 0.15)))
     )
@@
     (zone_connect 1)
     (attr smd)
-    (fp_text reference "D3" (at 0 2 180) (layer "F.SilkS")
+    (fp_text reference "D4" (at 0 2 180) (layer "F.SilkS")
         (effects (font (size 1 1) (thickness 0.15)))
     )
@@
     (property "ki_keywords" "R res resistor")
     (attr smd)
-    (fp_text reference "R14" (at 0 -1.3) (layer "F.SilkS")
+    (fp_text reference "R13" (at 0 -1.3) (layer "F.SilkS")
         (effects (font (size 0.8 0.8) (thickness 0.15)))
     )
@@
     (property "ki_keywords" "R res resistor")
     (attr smd)
-    (fp_text reference "R2" (at 0 -1.3) (layer "F.SilkS")
+    (fp_text reference "R12" (at 0 -1.3) (layer "F.SilkS")
         (effects (font (size 0.8 0.8) (thickness 0.15)))
     )
@@
     (property "ki_keywords" "R res resistor")
     (attr smd)
-    (fp_text reference "R6" (at 0 -1.3) (layer "F.SilkS")
+    (fp_text reference "R4" (at 0 -1.3) (layer "F.SilkS")
         (effects (font (size 0.8 0.8) (thickness 0.15)))
     )
@@
     (zone_connect 1)
     (attr smd)
-    (fp_text reference "C4" (at 0 -1.3) (layer "F.SilkS") hide
+    (fp_text reference "C1" (at 0 -1.3) (layer "F.SilkS") hide
         (effects (font (size 0.8 0.8) (thickness 0.15)))
     )
@@
     (property "ki_keywords" "R res resistor")
     (attr smd)
-    (fp_text reference "R13" (at 0 -1.3) (layer "F.SilkS")
+    (fp_text reference "R3" (at 0 -1.3) (layer "F.SilkS")
         (effects (font (size 0.8 0.8) (thickness 0.15)))
     )
@@
     (zone_connect 1)
     (attr smd)
-    (fp_text reference "C1" (at 0 -1.3) (layer "F.SilkS") hide
+    (fp_text reference "C8" (at 0 -1.3) (layer "F.SilkS") hide
         (effects (font (size 0.8 0.8) (thickness 0.15)))
     )
@@
     (property "ki_keywords" "R res resistor")
     (attr smd)
-    (fp_text reference "R15" (at 0 -1.3) (layer "F.SilkS")
+    (fp_text reference "R17" (at 0 -1.3) (layer "F.SilkS")
         (effects (font (size 0.8 0.8) (thickness 0.15)))
     )
@@
     (zone_connect 1)
     (attr smd)
-    (fp_text reference "C10" (at 0 -1.3) (layer "F.SilkS") hide
+    (fp_text reference "C6" (at 0 -1.3) (layer "F.SilkS") hide
         (effects (font (size 0.8 0.8) (thickness 0.15)))
     )
@@
     (zone_connect 1)
     (attr smd)
-    (fp_text reference "C2" (at 0 -1.3) (layer "F.SilkS") hide
+    (fp_text reference "C10" (at 0 -1.3) (layer "F.SilkS") hide
         (effects (font (size 0.8 0.8) (thickness 0.15)))
     )
@@
     (property "ki_keywords" "R res resistor")
     (attr smd)
-    (fp_text reference "R18" (at 0 -1.3) (layer "F.SilkS")
+    (fp_text reference "R16" (at 0 -1.3) (layer "F.SilkS")
         (effects (font (size 0.8 0.8) (thickness 0.15)))
     )
@@
     (property "ki_keywords" "R res resistor")
     (attr smd)
-    (fp_text reference "R11" (at 0 -1.3) (layer "F.SilkS")
+    (fp_text reference "R1" (at 0 -1.3) (layer "F.SilkS")
         (effects (font (size 0.8 0.8) (thickness 0.15)))
     )
@@
     (property "ki_keywords" "R res resistor")
     (attr smd)
-    (fp_text reference "R20" (at 0 -1.3) (layer "F.SilkS")
+    (fp_text reference "R14" (at 0 -1.3) (layer "F.SilkS")
         (effects (font (size 0.8 0.8) (thickness 0.15)))
     )
@@
     (zone_connect 1)
     (attr smd)
-    (fp_text reference "C7" (at 0 -1.3) (layer "F.SilkS") hide
+    (fp_text reference "C5" (at 0 -1.3) (layer "F.SilkS") hide
         (effects (font (size 0.8 0.8) (thickness 0.15)))
     )
@@
     (property "ki_keywords" "R res resistor")
     (attr smd)
-    (fp_text reference "R1" (at 0 -1.3) (layer "F.SilkS")
+    (fp_text reference "R7" (at 0 -1.3) (layer "F.SilkS")
         (effects (font (size 0.8 0.8) (thickness 0.15)))
     )
@@
     (zone_connect 1)
     (attr smd)
-    (fp_text reference "C5" (at 0 -1.3) (layer "F.SilkS") hide
+    (fp_text reference "C2" (at 0 -1.3) (layer "F.SilkS") hide
         (effects (font (size 0.8 0.8) (thickness 0.15)))
     )
@@
     (property "ki_keywords" "R res resistor")
     (attr smd)
-    (fp_text reference "R12" (at 0 -1.3) (layer "F.SilkS")
+    (fp_text reference "R2" (at 0 -1.3) (layer "F.SilkS")
         (effects (font (size 0.8 0.8) (thickness 0.15)))
     )
@@
     (property "ki_keywords" "R res resistor")
     (attr smd)
-    (fp_text reference "R7" (at 0 -1.3) (layer "F.SilkS")
+    (fp_text reference "R5" (at 0 -1.3) (layer "F.SilkS")
         (effects (font (size 0.8 0.8) (thickness 0.15)))
     )
@@
     (property "ki_keywords" "R res resistor")
     (attr smd)
-    (fp_text reference "R17" (at 0 -1.3) (layer "F.SilkS")
+    (fp_text reference "R18" (at 0 -1.3) (layer "F.SilkS")
         (effects (font (size 0.8 0.8) (thickness 0.15)))
     )
@@
     (property "ki_keywords" "R res resistor")
     (attr smd)
-    (fp_text reference "R16" (at 0 -1.3) (layer "F.SilkS")
+    (fp_text reference "R19" (at 0 -1.3) (layer "F.SilkS")
         (effects (font (size 0.8 0.8) (thickness 0.15)))
     )
@@
     (property "ki_keywords" "R res resistor")
     (attr smd)
-    (fp_text reference "R3" (at 0 -1.3) (layer "F.SilkS")
+    (fp_text reference "R9" (at 0 -1.3) (layer "F.SilkS")
         (effects (font (size 0.8 0.8) (thickness 0.15)))
     )
@@
     (property "ki_keywords" "R res resistor")
     (attr smd)
-    (fp_text reference "R8" (at 0 -1.3) (layer "F.SilkS")
+    (fp_text reference "R6" (at 0 -1.3) (layer "F.SilkS")
         (effects (font (size 0.8 0.8) (thickness 0.15)))
     )
@@
     (zone_connect 1)
     (attr smd)
-    (fp_text reference "D5" (at 0 2 180) (layer "F.SilkS")
+    (fp_text reference "D3" (at 0 2 180) (layer "F.SilkS")
         (effects (font (size 1 1) (thickness 0.15)))
     )
@@
     (zone_connect 1)
     (attr smd)
-    (fp_text reference "C3" (at 0 -1.3) (layer "F.SilkS") hide
+    (fp_text reference "C7" (at 0 -1.3) (layer "F.SilkS") hide
         (effects (font (size 0.8 0.8) (thickness 0.15)))
     )
@@
     (property "ki_keywords" "R res resistor")
     (attr smd)
-    (fp_text reference "R9" (at 0 -1.3) (layer "F.SilkS")
+    (fp_text reference "R11" (at 0 -1.3) (layer "F.SilkS")
         (effects (font (size 0.8 0.8) (thickness 0.15)))
     )
@@
     (zone_connect 1)
     (attr smd)
-    (fp_text reference "C6" (at 0 -1.3) (layer "F.SilkS") hide
+    (fp_text reference "C3" (at 0 -1.3) (layer "F.SilkS") hide
         (effects (font (size 0.8 0.8) (thickness 0.15)))
     )
@@
     (property "ki_keywords" "cap capacitor")
     (attr smd)
-    (fp_text reference "C9" (at 0 -1.9 180) (layer "F.SilkS")
-        (effects (font (size 0.8 0.8) (thickness 0.15)))
-    )
+    (fp_text reference "C4" (at 0 -1.9 180) (layer "F.SilkS")
+        (effects (font (size 0.8 0.8) (thickness 0.15)))
+    )

Commit message: Swap comparators for easier routing
Connections:
- R10 pad 2: Net-(U1B-+) -> Net-(U1D-+)
- R17 pad 1: Net-(R15-Pad1) -> Net-(R17-Pad1)
- R19 pad 1: Net-(R16-Pad1) -> Net-(R19-Pad1)
- R7 pad 2: Net-(U1A-+) -> Net-(U1B-+)
- R8 pad 2: Net-(U1B--) -> Net-(U1D--)
- R9 pad 2: Net-(U1A--) -> Net-(U1B--)
- U1 pad 1: /CHK0 -> /CHK1
- U1 pad 11: /CHK1 -> /CHK0
- U1 pad 13: Net-(R15-Pad1) -> Net-(R19-Pad1)
- U1 pad 14: Net-(R16-Pad1) -> /CHK0
- U1 pad 2: /CHK1 -> Net-(R17-Pad1)
- U1 pad 4: Net-(U1A--) -> /REF_D
- U1 pad 5: Net-(U1A-+) -> /CHK1
- U1 pad 8: /REF_D -> Net-(U1D--)
- U1 pad 9: /CHK0 -> Net-(U1D-+)
Changed lines of the file:
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@@
   (net 10 "Net-(D2-K)")
   (net 11 "Net-(D3-K)")
-  (net 12 "Net-(D5-K)")
-  (net 13 "Net-(U1A-+)")
-  (net 14 "/PROBE")
-  (net 15 "Net-(U1A--)")
-  (net 16 "Net-(U1B-+)")
-  (net 17 "/REF0")
-  (net 18 "Net-(U1B--)")
-  (net 19 "Net-(U2-ADJ)")
-  (net 20 "Net-(R15-Pad1)")
-  (net 21 "Net-(R16-Pad1)")
+  (net 12 "Net-(D4-K)")
+  (net 13 "/PROBE")
+  (net 14 "/REF0")
+  (net 15 "Net-(U2-ADJ)")
+  (net 16 "Net-(R17-Pad1)")
+  (net 17 "Net-(R19-Pad1)")
+  (net 18 "Net-(U1B-+)")
+  (net 19 "Net-(U1D--)")
+  (net 20 "Net-(U1B--)")
+  (net 21 "Net-(U1D-+)")
   (footprint "NevaDA:C_0402" (layer "F.Cu")
     (at 122.35 120)
@@
       (stroke (width 0.1) (type solid)) (layer "F.Fab"))
     (pad "1" smd rect (at -0.75 0) (size 0.8 0.9) (layers "F.Cu" "F.Paste" "F.Mask")
-      (net 14 "/PROBE") (pintype "passive"))
+      (net 13 "/PROBE") (pintype "passive"))
     (pad "2" smd rect (at 0.75 0) (size 0.8 0.9) (layers "F.Cu" "F.Paste" "F.Mask")
-      (net 16 "Net-(U1B-+)") (pintype "passive"))
+      (net 21 "Net-(U1D-+)") (pintype "passive"))
     (model "${KISYS3DMOD}/Resistor_SMD.3dshapes/R_0603_1608Metric.step"
       (offset (xyz 0 0 0))
@@
       (stroke (width 0.1) (type solid)) (layer "F.Fab"))
     (pad "1" smd rect (at -0.75 0) (size 0.8 0.9) (layers "F.Cu" "F.Paste" "F.Mask")
-      (net 17 "/REF0") (pintype "passive"))
+      (net 14 "/REF0") (pintype "passive"))
     (pad "2" smd rect (at 0.75 0) (size 0.8 0.9) (layers "F.Cu" "F.Paste" "F.Mask")
-      (net 18 "Net-(U1B--)") (pintype "passive"))
+      (net 19 "Net-(U1D--)") (pintype "passive"))
     (model "${KISYS3DMOD}/Resistor_SMD.3dshapes/R_0603_1608Metric.step"
       (offset (xyz 0 0 0))
@@
       (stroke (width 0.1) (type default)) (layer "F.Fab"))
     (pad "1" smd rect (at -1.3 0 180) (size 1.5 1.5) (layers "F.Cu" "F.Paste" "F.Mask")
-      (net 11 "Net-(D3-K)") (pinfunction "K") (pintype "passive"))
+      (net 12 "Net-(D4-K)") (pinfunction "K") (pintype "passive"))
     (pad "2" smd rect (at 1.3 0 180) (size 1.5 1.5) (layers "F.Cu" "F.Paste" "F.Mask")
       (net 8 "/VCC_REG") (pinfunction "A") (pintype "passive"))
@@
       (net 8 "/VCC_REG") (pintype "passive"))
     (pad "2" smd rect (at 0.75 0) (size 0.8 0.9) (layers "F.Cu" "F.Paste" "F.Mask")
-      (net 19 "Net-(U2-ADJ)") (pintype "passive"))
+      (net 15 "Net-(U2-ADJ)") (pintype "passive"))
     (model "${KISYS3DMOD}/Resistor_SMD.3dshapes/R_0603_1608Metric.step"
       (offset (xyz 0 0 0))
@@
       (net 6 "/REF1") (pintype "passive"))
     (pad "2" smd rect (at 0.75 0) (size 0.8 0.9) (layers "F.Cu" "F.Paste" "F.Mask")
-      (net 17 "/REF0") (pintype "passive"))
+      (net 14 "/REF0") (pintype "passive"))
     (model "${KISYS3DMOD}/Resistor_SMD.3dshapes/R_0603_1608Metric.step"
       (offset (xyz 0 0 0))
@@
       (net 5 "/CENTER") (pintype "passive"))
     (pad "2" smd rect (at 0.75 0) (size 0.8 0.9) (layers "F.Cu" "F.Paste" "F.Mask")
-      (net 14 "/PROBE") (pintype "passive"))
+      (net 13 "/PROBE") (pintype "passive"))
     (model "${KISYS3DMOD}/Resistor_SMD.3dshapes/R_0603_1608Metric.step"
       (offset (xyz 0 0 0))
@@
       (stroke (width 0.1) (type solid)) (layer "F.Fab"))
     (pad "1" smd rect (at -0.75 0) (size 0.8 0.9) (layers "F.Cu" "F.Paste" "F.Mask")
-      (net 20 "Net-(R15-Pad1)") (pintype "passive"))
+      (net 16 "Net-(R17-Pad1)") (pintype "passive"))
     (pad "2" smd rect (at 0.75 0) (size 0.8 0.9) (layers "F.Cu" "F.Paste" "F.Mask")
       (net 10 "Net-(D2-K)") (pintype "passive"))
@@
       (stroke (width 0.1) (type solid)) (layer "F.Fab"))
     (pad "1" smd rect (at -0.75 0) (size 0.8 0.9) (layers "F.Cu" "F.Paste" "F.Mask")
-      (net 19 "Net-(U2-ADJ)") (pintype "passive"))
+      (net 15 "Net-(U2-ADJ)") (pintype "passive"))
     (pad "2" smd rect (at 0.75 0) (size 0.8 0.9) (layers "F.Cu" "F.Paste" "F.Mask")
       (net 2 "GNDD") (pintype "passive"))
@@
       (stroke (width 0.15) (type solid)) (layer "F.Fab"))
     (pad "1" smd rect (at -3 -3.81 270) (size 2 0.6) (layers "F.Cu" "F.Paste" "F.Mask")
-      (net 4 "/CHK0") (pintype "open_collector"))
+      (net 1 "/CHK1") (pintype "open_collector"))
     (pad "2" smd rect (at -3 -2.54 270) (size 2 0.6) (layers "F.Cu" "F.Paste" "F.Mask")
-      (net 1 "/CHK1") (pintype "open_collector"))
+      (net 16 "Net-(R17-Pad1)") (pintype "open_collector"))
     (pad "3" smd rect (at -3 -1.27 270) (size 2 0.6) (layers "F.Cu" "F.Paste" "F.Mask")
       (net 7 "V+") (pinfunction "V+") (pintype "power_in"))
     (pad "4" smd rect (at -3 0 270) (size 2 0.6) (layers "F.Cu" "F.Paste" "F.Mask")
-      (net 15 "Net-(U1A--)") (pinfunction "-") (pintype "input"))
+      (net 3 "/REF_D") (pinfunction "-") (pintype "input"))
     (pad "5" smd rect (at -3 1.27 270) (size 2 0.6) (layers "F.Cu" "F.Paste" "F.Mask")
-      (net 13 "Net-(U1A-+)") (pinfunction "+") (pintype "input"))
+      (net 1 "/CHK1") (pinfunction "+") (pintype "input"))
     (pad "6" smd rect (at -3 2.54 270) (size 2 0.6) (layers "F.Cu" "F.Paste" "F.Mask")
-      (net 18 "Net-(U1B--)") (pinfunction "-") (pintype "input"))
+      (net 20 "Net-(U1B--)") (pinfunction "-") (pintype "input"))
     (pad "7" smd rect (at -3 3.81 270) (size 2 0.6) (layers "F.Cu" "F.Paste" "F.Mask")
-      (net 16 "Net-(U1B-+)") (pinfunction "+") (pintype "input"))
+      (net 18 "Net-(U1B-+)") (pinfunction "+") (pintype "input"))
     (pad "8" smd rect (at 3 3.81 270) (size 2 0.6) (layers "F.Cu" "F.Paste" "F.Mask")
-      (net 3 "/REF_D") (pinfunction "-") (pintype "input"))
+      (net 19 "Net-(U1D--)") (pinfunction "-") (pintype "input"))
     (pad "9" smd rect (at 3 2.54 270) (size 2 0.6) (layers "F.Cu" "F.Paste" "F.Mask")
-      (net 4 "/CHK0") (pinfunction "+") (pintype "input"))
+      (net 21 "Net-(U1D-+)") (pinfunction "+") (pintype "input"))
     (pad "10" smd rect (at 3 1.27 270) (size 2 0.6) (layers "F.Cu" "F.Paste" "F.Mask")
       (net 3 "/REF_D") (pinfunction "-") (pintype "input"))
     (pad "11" smd rect (at 3 0 270) (size 2 0.6) (layers "F.Cu" "F.Paste" "F.Mask")
-      (net 1 "/CHK1") (pinfunction "+") (pintype "input"))
+      (net 4 "/CHK0") (pinfunction "+") (pintype "input"))
     (pad "12" smd rect (at 3 -1.27 270) (size 2 0.6) (layers "F.Cu" "F.Paste" "F.Mask")
       (net 2 "GNDD") (pinfunction "V-") (pintype "power_in"))
     (pad "13" smd rect (at 3 -2.54 270) (size 2 0.6) (layers "F.Cu" "F.Paste" "F.Mask")
-      (net 20 "Net-(R15-Pad1)") (pintype "open_collector"))
+      (net 17 "Net-(R19-Pad1)") (pintype "open_collector"))
     (pad "14" smd rect (at 3 -3.81 270) (size 2 0.6) (layers "F.Cu" "F.Paste" "F.Mask")
-      (net 21 "Net-(R16-Pad1)") (pintype "open_collector"))
+      (net 4 "/CHK0") (pintype "open_collector"))
     (model "${KISYS3DMOD}/Package_SO.3dshapes/SOIC-14_3.9x8.7mm_P1.27mm.step"
       (offset (xyz 0 0 0))
@@
       (net 6 "/REF1") (pintype "passive"))
     (pad "2" smd rect (at 0.75 0) (size 0.8 0.9) (layers "F.Cu" "F.Paste" "F.Mask")
-      (net 13 "Net-(U1A-+)") (pintype "passive"))
+      (net 18 "Net-(U1B-+)") (pintype "passive"))
     (model "${KISYS3DMOD}/Resistor_SMD.3dshapes/R_0603_1608Metric.step"
       (offset (xyz 0 0 0))
@@
       (net 2 "GNDD") (pintype "passive"))
     (pad "2" smd rect (at 0.75 0) (size 0.8 0.9) (layers "F.Cu" "F.Paste" "F.Mask")
-      (net 12 "Net-(D5-K)") (pintype "passive"))
+      (net 11 "Net-(D3-K)") (pintype "passive"))
     (model "${KISYS3DMOD}/Resistor_SMD.3dshapes/R_0603_1608Metric.step"
       (offset (xyz 0 0 0))
@@
       (stroke (width 0.1) (type solid)) (layer "F.Fab"))
     (pad "1" smd rect (at -0.75 0) (size 0.8 0.9) (layers "F.Cu" "F.Paste" "F.Mask")
-      (net 21 "Net-(R16-Pad1)") (pintype "passive"))
+      (net 17 "Net-(R19-Pad1)") (pintype "passive"))
     (pad "2" smd rect (at 0.75 0) (size 0.8 0.9) (layers "F.Cu" "F.Paste" "F.Mask")
-      (net 11 "Net-(D3-K)") (pintype "passive"))
+      (net 12 "Net-(D4-K)") (pintype "passive"))
     (model "${KISYS3DMOD}/Resistor_SMD.3dshapes/R_0603_1608Metric.step"
       (offset (xyz 0 0 0))
@@
       (stroke (width 0.1) (type solid)) (layer "F.Fab"))
     (pad "1" smd rect (at -0.75 0) (size 0.8 0.9) (layers "F.Cu" "F.Paste" "F.Mask")
-      (net 14 "/PROBE") (pintype "passive"))
+      (net 13 "/PROBE") (pintype "passive"))
     (pad "2" smd rect (at 0.75 0) (size 0.8 0.9) (layers "F.Cu" "F.Paste" "F.Mask")
-      (net 15 "Net-(U1A--)") (pintype "passive"))
+      (net 20 "Net-(U1B--)") (pintype "passive"))
     (model "${KISYS3DMOD}/Resistor_SMD.3dshapes/R_0603_1608Metric.step"
       (offset (xyz 0 0 0))
@@
       (stroke (width 0.1) (type solid)) (layer "F.Fab"))
     (pad "1" smd rect (at -0.75 0) (size 0.8 0.9) (layers "F.Cu" "F.Paste" "F.Mask")
-      (net 17 "/REF0") (pintype "passive"))
+      (net 14 "/REF0") (pintype "passive"))
     (pad "2" smd rect (at 0.75 0) (size 0.8 0.9) (layers "F.Cu" "F.Paste" "F.Mask")
       (net 2 "GNDD") (pintype "passive"))
@@
     (pad "" smd rect (at 3.775 1.525) (size 3.05 2.75) (layers "F.Paste"))
     (pad "1" smd rect (at -4.2 -2.28) (size 2.2 1.2) (layers "F.Cu" "F.Paste" "F.Mask")
-      (net 19 "Net-(U2-ADJ)") (pinfunction "ADJ") (pintype "input"))
+      (net 15 "Net-(U2-ADJ)") (pinfunction "ADJ") (pintype "input"))
     (pad "2" smd rect (at 2.1 0) (size 6.4 5.8) (layers "F.Cu" "F.Mask")
       (net 8 "/VCC_REG") (pinfunction "VO") (pintype "power_out") (zone_connect 2))
@@
       (stroke (width 0.1) (type default)) (layer "F.Fab"))
     (pad "1" smd rect (at -1.3 0 180) (size 1.5 1.5) (layers "F.Cu" "F.Paste" "F.Mask")
-      (net 12 "Net-(D5-K)") (pinfunction "K") (pintype "passive"))
+      (net 11 "Net-(D3-K)") (pinfunction "K") (pintype "passive"))
     (pad "2" smd rect (at 1.3 0 180) (size 1.5 1.5) (layers "F.Cu" "F.Paste" "F.Mask")
       (net 8 "/VCC_REG") (pinfunction "A") (pintype "passive"))

Commit message: Input circuits layout stub
Parts:
- moved C1 56.1 mm to (89.0, 99.0)
- moved R1 50.3 mm to (87.2, 96.8), turned to -90 degrees
- moved R2 49.9 mm to (87.2, 103.2), turned to -90 degrees
- moved R3 44.4 mm to (87.2, 100.0), turned to -90 degrees
- moved C2 36.9 mm to (89.0, 97.0), turned to 180 degrees
- moved R4 34.2 mm to (90.8, 100.0), turned to -90 degrees
- moved R5 33.2 mm to (90.8, 96.8), turned to -90 degrees
- moved R6 33.1 mm to (90.8, 103.2), turned to -90 degrees
- moved R8 16.9 mm to (93.2, 103.0)
- moved R7 15.8 mm to (93.2, 97.0)
- moved R10 15.5 mm to (93.2, 101.0)
- moved R9 15.3 mm to (93.2, 99.0)
