File: logic_tester.kicad_sch (KiCad schematic)
At the start: 37 parts, among them J1 15EDGR-3.5-02P, J2 Probe, U1 LM339D, U2 LM317MDT

Commit message: Title added to sheets
Other:
- company: (none) -> OSHW
- title: (none) -> Logic tester
Changed lines of the file:
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@@
 (kicad_sch (version 20230121) (generator eeschema)
   (paper "A4")
+  (title_block
+    (title "Logic tester")
+    (date "2024-11-23")
+    (rev "1.0")
+    (company "OSHW")
+  )
   (junction (at 215.9 88.9) (diameter 0) (color 0 0 0 0)
   )
